File: ECAD/PCBs/Functional PCBs/UFC_Main/UFC_Main.kicad_pcb (KiCad board)
At the start: 2 copper layers, 168 x 110 mm, 255 parts, among them J1 EXT_PWR, J10 GPIO3, J11 GPIO2, J12 AIN3, J13 5V I2C, J2 ENC1, J3 VOL1, J4 BRT, J5 AP KB, J6 HUD BIT, J7 ENC2, J8 VOL2, J9 ADF SW, Q2 2N7002, Q4 SKML5203, Q5 SI2302, Q6 SKML5203, Q7 SKML5203, Q8 SI2302, SW1 B3F-1026, SW10 B3F-1026, SW11 B3F-1026, SW12 B3F-1026, SW13 B3F-1026, SW14 B3F-1026, SW15 B3F-1026, SW16 B3F-1026, SW17 B3F-1026, SW18 B3F-1026, SW19 B3F-1026, SW2 B3F-1026, SW3 B3F-1026, SW4 B3F-1026, SW5 B3F-1026, SW6 B3F-1026, SW7 B3F-1026, SW8 B3F-1026, SW9 B3F-1026, U1 HT1621B, U10 TCA8418RTWR, U11 GN1640T, U12 GN1640T, U13 ADS1115IDGSR, U14 ADR5040ARTZ, U2 GN1640T, U3 GN1640T, U4 GN1640T, U5 GN1640T, U6 GN1640T, U7 GN1640T, U8 TXS0108EPWR, U9 TXS0108EPWR

Commit message: 1181# Update ECAD source files
Updated ECAD source files for UFC Main V6.3.1.
Parts:
- added R16: 4.7K, Resistor_SMD:R_0603_1608Metric, B.Cu at (113.8, 169.9)
- added R17: 4.7K, Resistor_SMD:R_0603_1608Metric, B.Cu at (120.5, 176.8)
- added R18: 4.7k, Resistor_SMD:R_0603_1608Metric, B.Cu at (155.1, 196.4)
- DS2, DS3, DS4, DS5, DS6: footprint OH_Footprints:UFCOptionDigitV3 -> Socket:UFCOptionDigitV3RectanglePads
- moved C19 0.43 mm to (114.0, 172.2)
- moved C18 0.43 mm to (112.8, 172.2)
Connections:
- U13 pad 1: GND -> Net-(U13-ADDR)
Routing:
- net GND: track 260.3 -> 274.1 mm
- net +3V3: track 232.8 -> 239.4 mm
- net IO_INT: track 10.5 -> 13.3 mm
- net Net-(U13-ADDR): track 0.00 -> 1.81 mm
- net ADC_RDY@3.3V: track 17.2 -> 18.3 mm
- net /AIN0: track 17.7 -> 18.6 mm
- net Net-(J12-Pin_1): track 7.91 -> 8.64 mm
- net COM2_CLK: track 136.3 -> 135.8 mm
