File: ECAD/PCBs/Functional PCBs/UFC_Main/UFC_Main.kicad_sch (KiCad schematic)
At the start: 253 parts, among them J1 EXT_PWR, J10 GPIO3, J11 GPIO2, J12 AIN3, J13 5V I2C, J2 ENC1, J3 VOL1, J4 BRT, J5 AP KB, J6 HUD BIT, J7 ENC2, J8 VOL2, J9 ADF SW, Q2 2N7002, Q4 SKML5203, Q5 SI2302, Q6 SKML5203, Q7 SKML5203, Q8 SI2302, SW1 B3F-1026, U1 HT1621B, U10 TCA8418RTWR, U11 GN1640T, U12 GN1640T, U13 ADS1115IDGSR, U14 ADR5040ARTZ, U2 GN1640T, U3 GN1640T, U4 GN1640T, U5 GN1640T, U6 GN1640T, U7 GN1640T, U8 TXS0108EPWR, U9 TXS0108EPWR

Commit message: 1181# Update ECAD source files
Updated ECAD source files for UFC Main V6.3.1.
Parts:
- added R16, R17: 4.7K, Resistor_SMD:R_0603_1608Metric, symbol Device:R_Small
- added R18: 4.7k, Resistor_SMD:R_0603_1608Metric, symbol Device:R_Small
- renumbered C1 to C14, D23 to D100, D24 to D101, D9 to D102, D10 to D103, D11 to D104, D12 to D105, D13 to D106, D14 to D107, D15 to D108, D16 to D109, D17 to D110, D18 to D111, D19 to D112, D20 to D113, D21 to D114, D22 to D115, D23 to D116, D24 to D117, D1 to D25, D2 to D26, D3 to D27, D4 to D28, D5 to D29, D6 to D30, D7 to D31, D8 to D32, D9 to D33, D10 to D34, D11 to D35, D12 to D36, D13 to D41, D14 to D42, D15 to D43, D16 to D44, D17 to D45, D18 to D46, D19 to D47, D20 to D48, D21 to D49, D22 to D50, D23 to D51, D24 to D52, D9 to D53, D10 to D54, D11 to D55, D12 to D56, D13 to D57, D14 to D58, D15 to D59, D16 to D60, D17 to D61, D18 to D62, D19 to D63, D20 to D64, D21 to D65, D22 to D66, D23 to D67, D24 to D68, D9 to D86, D10 to D87, D11 to D88, D12 to D89, D13 to D90, D14 to D91, D15 to D92, D16 to D93, D17 to D94, D18 to D95, D19 to D96, D20 to D97, D21 to D98, D22 to D99, SW1 to SW10, SW1 to SW11, SW1 to SW12, SW1 to SW13, SW1 to SW14, SW1 to SW15, SW1 to SW16, SW1 to SW17, SW1 to SW18, SW1 to SW19, SW1 to SW2, SW1 to SW3, SW1 to SW4, SW1 to SW5, SW1 to SW6, SW1 to SW7, SW1 to SW8, SW1 to SW9
Connections:
- net +3V3: now also R17.1, R18.1
- net ADC_RDY@3.3V: now also R17.2
- net GND: now also R16.2; no longer U13.1 (ADDR)
- net IO_INT: now also R18.2
- new net: R16.1, U13.1 (ADDR)
Other:
- note added: "GPIO EXPANDER"
- moved on the sheet: R10, R4, R9
